File: macropad1.sch (KiCad schematic (older format))
At the start: 18 parts, among them J1 Conn_01x04, SW1 SW_Reed, SW2 Rotary_Encoder_Switch, U1 ATmega32U4-AU, Y1 16Mhz

Commit message: Ready for prototyping
Parts:
- removed USB1: Molex-0548190589, random-keyboard-parts:Molex-0548190589, symbol random-keyboard-parts:Molex-0548190589
- added J2: USB_B_Mini, Connector_USB:USB_Mini-B_Lumberg_2486_01_Horizontal, symbol Connector:USB_B_Mini
Connections:
- wire segments 78 -> 73
- no-connect marks 13 -> 14
Other:
- moved on the sheet: F1
Changed lines of the file:
@@
 Comment4 ""
 $EndDescr
-$Comp
-L power:+5V #PWR0101
-U 1 1 5F42D04E
-P 3800 1750
-F 0 "#PWR0101" H 3800 1600 50  0001 C CNN
-F 1 "+5V" H 3815 1923 50  0000 C CNN
-F 2 "" H 3800 1750 50  0001 C CNN
-F 3 "" H 3800 1750 50  0001 C CNN
-	1    3800 1750
-	1    0    0    -1
-$EndComp
 Wire Wire Line
 	4000 1900 3900 1900
@@
 $EndComp
 $Comp
-L power:+5V #PWR0105
-U 1 1 5F43A2D6
-P 1400 3800
-F 0 "#PWR0105" H 1400 3650 50  0001 C CNN
-F 1 "+5V" H 1415 3973 50  0000 C CNN
-F 2 "" H 1400 3800 50  0001 C CNN
-F 3 "" H 1400 3800 50  0001 C CNN
-	1    1400 3800
-	1    0    0    -1
-$EndComp
-$Comp
 L power:GND #PWR0106
 U 1 1 5F43A770
@@
 	800  4000 1200 4000
 Connection ~ 1200 4000
-Wire Wire Line
-	1200 4000 1400 4000
 Connection ~ 1600 4000
 Wire Wire Line
@@
 	1600 4200 1400 4200
 Wire Wire Line
-	1400 3800 1400 4000
-Connection ~ 1400 4000
-Wire Wire Line
-	1400 4000 1600 4000
-Wire Wire Line
 	1400 4300 1400 4200
 Connection ~ 1400 4200
 Wire Wire Line
 	1400 4200 1200 4200
-$Comp
-L power:+5V #PWR0107
-U 1 1 5F43C6D6
-P 1300 2950
-F 0 "#PWR0107" H 1300 2800 50  0001 C CNN
-F 1 "+5V" H 1315 3123 50  0000 C CNN
-F 2 "" H 1300 2950 50  0001 C CNN
-F 3 "" H 1300 2950 50  0001 C CNN
-	1    1300 2950
-	1    0    0    -1
-$EndComp
-Wire Wire Line
-	3300 3000 1300 3000
-Wire Wire Line
-	1300 3000 1300 2950
 $Comp
 L Device:Crystal_GND24_Small Y1
@@
 	2550 1750 2250 1750
 $Comp
-L power:+5V #PWR0110
-U 1 1 5F4696D9
-P 2950 1200
-F 0 "#PWR0110" H 2950 1050 50  0001 C CNN
-F 1 "+5V" H 2965 1373 50  0000 C CNN
-F 2 "" H 2950 1200 50  0001 C CNN
-F 3 "" H 2950 1200 50  0001 C CNN
-	1    2950 1200
-	1    0    0    -1
-$EndComp
-$Comp
 L Device:R_Small_US R4
 U 1 1 5F46A1EB
@@
 L Device:Polyfuse_Small F1
 U 1 1 5F4711D6
-P 8700 2350
-F 0 "F1" V 8495 2350 50  0000 C CNN
-F 1 "500mA" V 8586 2350 50  0000 C CNN
-F 2 "Fuse:Fuse_1206_3216Metric" H 8750 2150 50  0001 L CNN
-F 3 "~" H 8700 2350 50  0001 C CNN
-	1    8700 2350
+P 8600 3450
+F 0 "F1" V 8395 3450 50  0000 C CNN
+F 1 "500mA" V 8486 3450 50  0000 C CNN
+F 2 "Fuse:Fuse_1206_3216Metric" H 8650 3250 50  0001 L CNN
+F 3 "~" H 8600 3450 50  0001 C CNN
+	1    8600 3450
 	0    1    1    0
 $EndComp
 Wire Wire Line
-	7750 2350 8250 2350
-$Comp
-L power:+5V #PWR0111
-U 1 1 5F4757AD
-P 9300 2300
-F 0 "#PWR0111" H 9300 2150 50  0001 C CNN
-F 1 "+5V" H 9315 2473 50  0000 C CNN
-F 2 "" H 9300 2300 50  0001 C CNN
-F 3 "" H 9300 2300 50  0001 C CNN
-	1    9300 2300
-	1    0    0    -1
-$EndComp
-Wire Wire Line
-	9300 2300 9300 2350
-Wire Wire Line
-	9300 2350 8800 2350
+	7650 3450 8150 3450
+Wire Wire Line
+	9200 3450 8700 3450
 $Comp
 L power:VCC #PWR0112
 U 1 1 5F476F4F
-P 8250 2300
-F 0 "#PWR0112" H 8250 2150 50  0001 C CNN
-F 1 "VCC" H 8265 2473 50  0000 C CNN
-F 2 "" H 8250 2300 50  0001 C CNN
-F 3 "" H 8250 2300 50  0001 C CNN
-	1    8250 2300
-	1    0    0    -1
-$EndComp
-Wire Wire Line
-	8250 2300 8250 2350
-Connection ~ 8250 2350
-Wire Wire Line
-	8250 2350 8600 2350
-Text GLabel 8050 2550 2    50   Input ~ 0
+P 8150 3400
+F 0 "#PWR0112" H 8150 3250 50  0001 C CNN
+F 1 "VCC" H 8165 3573 50  0000 C CNN
+F 2 "" H 8150 3400 50  0001 C CNN
+F 3 "" H 8150 3400 50  0001 C CNN
+	1    8150 3400
+	1    0    0    -1
+$EndComp
+Wire Wire Line
+	8150 3400 8150 3450
+Connection ~ 8150 3450
+Wire Wire Line
+	8150 3450 8500 3450
+Text GLabel 7750 3750 2    50   Input ~ 0
 D+
-Text GLabel 8050 2450 2    50   Input ~ 0
+Text GLabel 7750 3650 2    50   Input ~ 0
 D-
-Wire Wire Line
-	8050 2450 7750 2450
-Wire Wire Line
-	7750 2550 8050 2550
 $Comp
 L power:GND #PWR0113
 U 1 1 5F47A741
-P 8050 2850
-F 0 "#PWR0113" H 8050 2600 50  0001 C CNN
-F 1 "GND" H 8055 2677 50  0000 C CNN
-F 2 "" H 8050 2850 50  0001 C CNN
-F 3 "" H 8050 2850 50  0001 C CNN
-	1    8050 2850
-	1    0    0    -1
-$EndComp
-Wire Wire Line
-	8050 2850 8050 2750
-Wire Wire Line
-	8050 2750 7900 2750
+P 7250 4250
+F 0 "#PWR0113" H 7250 4000 50  0001 C CNN
+F 1 "GND" H 7255 4077 50  0000 C CNN
+F 2 "" H 7250 4250 50  0001 C CNN
+F 3 "" H 7250 4250 50  0001 C CNN
+	1    7250 4250
+	1    0    0    -1
+$EndComp
 $Sheet
 S 10100 800  600  1650
@@
 SDA
 Wire Wire Line
-	7750 2250 7900 2250
-Wire Wire Line
-	7900 2250 7900 2750
-Connection ~ 7900 2750
-Wire Wire Line
-	7900 2750 7750 2750
-$Comp
-L random-keyboard-parts:Molex-0548190589 USB1
-U 1 1 5F4707AD
-P 7450 2550
-F 0 "USB1" V 7987 2517 60  0000 C CNN
-F 1 "Molex-0548190589" V 7881 2517 60  0000 C CNN
-F 2 "random-keyboard-parts:Molex-0548190589" H 7450 2550 60  0001 C CNN
-F 3 "" H 7450 2550 60  0001 C CNN
-	1    7450 2550
-	0    -1   -1   0
-$EndComp
-NoConn ~ 7750 2650
-Wire Wire Line
 	5250 3750 4900 3750
 Wire Wire Line
@@
 Text Label 4500 3400 0    50   ~ 0
 SCL
-$Comp
-L power:+5V #PWR0114
-U 1 1 5F5F59A8
-P 5700 3600
-F 0 "#PWR0114" H 5700 3450 50  0001 C CNN
-F 1 "+5V" H 5715 3773 50  0000 C CNN
-F 2 "" H 5700 3600 50  0001 C CNN
-F 3 "" H 5700 3600 50  0001 C CNN
-	1    5700 3600
-	1    0    0    -1
-$EndComp
 Wire Wire Line
 	5700 3600 6050 3600
@@
 	1    0    0    -1
 $EndComp
-$Comp
-L power:GND #PWR0115
-U 1 1 5F606F2E
-P 10350 4600
-F 0 "#PWR0115" H 10350 4350 50  0001 C CNN
-F 1 "GND" H 10355 4427 50  0000 C CNN
-F 2 "" H 10350 4600 50  0001 C CNN
-F 3 "" H 10350 4600 50  0001 C CNN
-	1    10350 4600
-	1    0    0    -1
-$EndComp
 Text Label 6300 1450 0    50   ~ 0
 ENC_S1
 Text Label 6300 1650 0    50   ~ 0
 ENC_S2
-Text Label 10350 4500 0    50   ~ 0
-GND
-Wire Wire Line
-	10350 4500 10350 4600
 Text Label 5550 1550 2    50   ~ 0
 GND
@@
 Wire Wire Line
 	6200 1650 6300 1650
+$Comp
+L Connector:USB_B_Mini J2
+U 1 1 5F4CA438
+P 7350 3650
+F 0 "J2" H 7407 4117 50  0000 C CNN
+F 1 "USB_B_Mini" H 7407 4026 50  0000 C CNN
+F 2 "Connector_USB:USB_Mini-B_Lumberg_2486_01_Horizontal" H 7500 3600 50  0001 C CNN
+F 3 "~" H 7500 3600 50  0001 C CNN
+	1    7350 3650
+	1    0    0    -1
+$EndComp
+Wire Wire Line
+	7350 4050 7250 4050
+Wire Wire Line
+	7250 4050 7250 4250
+Wire Wire Line
+	7750 3650 7650 3650
+Wire Wire Line
+	7750 3750 7650 3750
+Connection ~ 7250 4050
+NoConn ~ 7650 3850
+NoConn ~ 3300 2800
+Wire Wire Line
+	3300 3000 1150 3000
+Wire Wire Line
+	1150 3000 1150 2600
+Wire Wire Line
+	1200 4000 1400 4000
+Wire Wire Line
+	1400 3900 1400 4000
+Connection ~ 1400 4000
+Wire Wire Line
+	1400 4000 1600 4000
+$Comp
+L power:PWR_FLAG #FLG0101
+U 1 1 5F4D9E9A
+P 1850 6150
+F 0 "#FLG0101" H 1850 6225 50  0001 C CNN
+F 1 "PWR_FLAG" H 1850 6323 50  0000 C CNN
+F 2 "" H 1850 6150 50  0001 C CNN
+F 3 "~" H 1850 6150 50  0001 C CNN
+	1    1850 6150
+	-1   0    0    1
+$EndComp
+$Comp
+L power:+5V #PWR0101
+U 1 1 5F4DCBB7
+P 1850 6150
+F 0 "#PWR0101" H 1850 6000 50  0001 C CNN
+F 1 "+5V" H 1865 6323 50  0000 C CNN
+F 2 "" H 1850 6150 50  0001 C CNN
+F 3 "" H 1850 6150 50  0001 C CNN
+	1    1850 6150
+	1    0    0    -1
+$EndComp
+$Comp
+L power:+5V #PWR0105
+U 1 1 5F4DD150
+P 1400 3900
+F 0 "#PWR0105" H 1400 3750 50  0001 C CNN
+F 1 "+5V" H 1415 4073 50  0000 C CNN
+F 2 "" H 1400 3900 50  0001 C CNN
+F 3 "" H 1400 3900 50  0001 C CNN
+	1    1400 3900
+	1    0    0    -1
+$EndComp
+$Comp
+L power:+5V #PWR0107
+U 1 1 5F4DD7D3
+P 1150 2600
+F 0 "#PWR0107" H 1150 2450 50  0001 C CNN
+F 1 "+5V" H 1165 2773 50  0000 C CNN
+F 2 "" H 1150 2600 50  0001 C CNN
+F 3 "" H 1150 2600 50  0001 C CNN
+	1    1150 2600
+	1    0    0    -1
+$EndComp
+$Comp
+L power:+5V #PWR0110
+U 1 1 5F4DDBFF
+P 3800 1750
+F 0 "#PWR0110" H 3800 1600 50  0001 C CNN
+F 1 "+5V" H 3815 1923 50  0000 C CNN
+F 2 "" H 3800 1750 50  0001 C CNN
+F 3 "" H 3800 1750 50  0001 C CNN
+	1    3800 1750
+	1    0    0    -1
+$EndComp
+$Comp
+L power:+5V #PWR0111
+U 1 1 5F4DE0DF
+P 9200 3450
+F 0 "#PWR0111" H 9200 3300 50  0001 C CNN
+F 1 "+5V" H 9215 3623 50  0000 C CNN
+F 2 "" H 9200 3450 50  0001 C CNN
+F 3 "" H 9200 3450 50  0001 C CNN
+	1    9200 3450
+	1    0    0    -1
+$EndComp
+$Comp
+L power:+5V #PWR0114
+U 1 1 5F4DE8FE
+P 2950 1200
+F 0 "#PWR0114" H 2950 1050 50  0001 C CNN
+F 1 "+5V" H 2965 1373 50  0000 C CNN
+F 2 "" H 2950 1200 50  0001 C CNN
+F 3 "" H 2950 1200 50  0001 C CNN
+	1    2950 1200
+	1    0    0    -1
+$EndComp
+$Comp
+L power:+5V #PWR0116
+U 1 1 5F4E061A
+P 5700 3600
+F 0 "#PWR0116" H 5700 3450 50  0001 C CNN
+F 1 "+5V" H 5715 3773 50  0000 C CNN
+F 2 "" H 5700 3600 50  0001 C CNN
+F 3 "" H 5700 3600 50  0001 C CNN
+	1    5700 3600
+	1    0    0    -1
+$EndComp
 $EndSCHEMATC

Commit message: Added artwork lib and eeprom
Parts:
- added U2: 24LC512, Package_SO:TSSOP-8_4.4x3mm_P0.65mm, symbol Memory_EEPROM:24LC512
Connections:
- net +5V: now also U2.8 (VCC)
- net GND: now also U2.1 (A0), U2.2 (A1), U2.3 (A2), U2.4 (GND), U2.7 (WP)
- net SCL: now also U2.6 (SCL)
- net SDA: now also U2.5 (SDA)
Changed lines of the file:
@@
 	1    0    0    -1
 $EndComp
+$Comp
+L Memory_EEPROM:24LC512 U2
+U 1 1 5F50FB6A
+P 7850 1600
+F 0 "U2" H 7850 2081 50  0000 C CNN
+F 1 "24LC512" H 7850 1990 50  0000 C CNN
+F 2 "Package_SO:TSSOP-8_4.4x3mm_P0.65mm" H 7850 1600 50  0001 C CNN
+F 3 "http://ww1.microchip.com/downloads/en/DeviceDoc/21754M.pdf" H 7850 1600 50  0001 C CNN
+	1    7850 1600
+	1    0    0    -1
+$EndComp
+Text Label 8250 1600 0    50   ~ 0
+SCL
+Text Label 8250 1500 0    50   ~ 0
+SDA
+Wire Wire Line
+	7450 1500 7400 1500
+Wire Wire Line
+	7400 1500 7400 1600
+$Comp
+L power:GND #PWR0115
+U 1 1 5F51AA52
+P 7400 2150
+F 0 "#PWR0115" H 7400 1900 50  0001 C CNN
+F 1 "GND" H 7405 1977 50  0000 C CNN
+F 2 "" H 7400 2150 50  0001 C CNN
+F 3 "" H 7400 2150 50  0001 C CNN
+	1    7400 2150
+	1    0    0    -1
+$EndComp
+Wire Wire Line
+	7450 1700 7400 1700
+Connection ~ 7400 1700
+Wire Wire Line
+	7450 1600 7400 1600
+Connection ~ 7400 1600
+Wire Wire Line
+	7400 1600 7400 1700
+Wire Wire Line
+	7400 1700 7400 1900
+Wire Wire Line
+	7850 1900 7400 1900
+Connection ~ 7400 1900
+Wire Wire Line
+	7400 1900 7400 2150
+$Comp
+L power:+5V #PWR0117
+U 1 1 5F52923E
+P 8150 1250
+F 0 "#PWR0117" H 8150 1100 50  0001 C CNN
+F 1 "+5V" H 8165 1423 50  0000 C CNN
+F 2 "" H 8150 1250 50  0001 C CNN
+F 3 "" H 8150 1250 50  0001 C CNN
+	1    8150 1250
+	1    0    0    -1
+$EndComp
+Wire Wire Line
+	7850 1300 8150 1300
+Wire Wire Line
+	8150 1300 8150 1250
+Wire Wire Line
+	8250 1700 8250 1900
+Wire Wire Line
+	8250 1900 7850 1900
+Connection ~ 7850 1900
 $EndSCHEMATC

Commit message: Fixes D+/D- swap and adds ISP header
Also moves some components around for better layout
Parts:
- removed SW1: SW_Reed, Button_Switch_SMD:SW_SPST_REED_CT05-XXXX-G1, symbol Switch:SW_Reed
- added J3: AVR-ISP-6, Connector_PinHeader_2.54mm:PinHeader_2x03_P2.54mm_Vertical, symbol Connector:AVR-ISP-6
- added SW1: SPST, Button_Switch_SMD:SW_SPST_REED_CT05-XXXX-G1, symbol tinkerforge:SPST
Connections:
- net +5V: now also J3.2 (VCC)
- net D+: now also R2.1, U1.4 (D+); no longer J2.2 (D-), R2.2
- net D-: now also U1.3 (D-); no longer J2.3 (D+)
- net ENC_S1: now also J3.1 (MISO)
- net ENC_S2: now also J3.4 (MOSI)
- net GND: now also J3.6 (GND), SW1.1
- net RE_B: now also J3.3 (SCK)
- net !RESET: now reaches R4.2, U1.13 (~RESET)
- net !RESET: now also J3.5 (~RST), SW1.2
- net at R3.1: now also J2.2 (D-); no longer U1.3 (D-)
- new net: J2.3 (D+), R2.2
Other:
- moved on the sheet: R2, R3
Changed lines of the file:
@@
 L Device:R_Small_US R3
 U 1 1 5F432C2C
-P 2650 3300
-F 0 "R3" V 2445 3300 50  0000 C CNN
-F 1 "22" V 2536 3300 50  0000 C CNN
-F 2 "Resistor_SMD:R_0805_2012Metric" H 2650 3300 50  0001 C CNN
-F 3 "~" H 2650 3300 50  0001 C CNN
-	1    2650 3300
-	0    1    1    0
+P 7850 3750
+F 0 "R3" V 7645 3750 50  0000 C CNN
+F 1 "22" V 7736 3750 50  0000 C CNN
+F 2 "Resistor_SMD:R_0805_2012Metric" H 7850 3750 50  0001 C CNN
+F 3 "~" H 7850 3750 50  0001 C CNN
+	1    7850 3750
+	0    -1   -1   0
 $EndComp
 $Comp
 L Device:R_Small_US R2
 U 1 1 5F4331FA
-P 2300 3200
-F 0 "R2" V 2095 3200 50  0000 C CNN
-F 1 "22" V 2186 3200 50  0000 C CNN
-F 2 "Resistor_SMD:R_0805_2012Metric" H 2300 3200 50  0001 C CNN
-F 3 "~" H 2300 3200 50  0001 C CNN
-	1    2300 3200
+P 7850 3650
+F 0 "R2" V 7645 3650 50  0000 C CNN
+F 1 "22" V 7736 3650 50  0000 C CNN
+F 2 "Resistor_SMD:R_0805_2012Metric" H 7850 3650 50  0001 C CNN
+F 3 "~" H 7850 3650 50  0001 C CNN
+	1    7850 3650
 	0    1    1    0
 $EndComp
 Wire Wire Line
-	3300 3300 2750 3300
-Wire Wire Line
 	2400 3200 3300 3200
-Wire Wire Line
-	2200 3200 1300 3200
-Wire Wire Line
-	2550 3300 1300 3300
 $Comp
 L Device:C_Small C1
@@
 Connection ~ 1800 2750
 $Comp
-L Switch:SW_Reed SW1
-U 1 1 5F466CA0
-P 2750 1750
-F 0 "SW1" H 2750 1972 50  0000 C CNN
-F 1 "SW_Reed" H 2750 1881 50  0000 C CNN
-F 2 "Button_Switch_SMD:SW_SPST_REED_CT05-XXXX-G1" H 2750 1750 50  0001 C CNN
-F 3 "~" H 2750 1750 50  0001 C CNN
-	1    2750 1750
-	1    0    0    -1
-$EndComp
-$Comp
 L power:GND #PWR0109
 U 1 1 5F467A70
-P 2250 1750
-F 0 "#PWR0109" H 2250 1500 50  0001 C CNN
-F 1 "GND" H 2255 1577 50  0000 C CNN
-F 2 "" H 2250 1750 50  0001 C CNN
-F 3 "" H 2250 1750 50  0001 C CNN
-	1    2250 1750
-	1    0    0    -1
-$EndComp
-Wire Wire Line
-	3300 2200 2950 2200
-Wire Wire Line
-	2950 2200 2950 1750
-Connection ~ 2950 1750
-Wire Wire Line
-	2950 1750 2950 1500
-Wire Wire Line
-	2550 1750 2250 1750
+P 1450 1800
+F 0 "#PWR0109" H 1450 1550 50  0001 C CNN
+F 1 "GND" H 1455 1627 50  0000 C CNN
+F 2 "" H 1450 1800 50  0001 C CNN
+F 3 "" H 1450 1800 50  0001 C CNN
+	1    1450 1800
+	1    0    0    -1
+$EndComp
+Wire Wire Line
+	1950 1800 1450 1800
 $Comp
 L Device:R_Small_US R4
@@
 Wire Wire Line
 	2950 1200 2950 1300
-Text GLabel 1300 3200 0    50   Input ~ 0
+Text GLabel 2400 3200 0    50   Input ~ 0
 D+
-Text GLabel 1300 3300 0    50   Input ~ 0
+Text GLabel 2400 3300 0    50   Input ~ 0
 D-
 $Comp
@@
 Wire Wire Line
 	8150 3450 8500 3450
-Text GLabel 7750 3750 2    50   Input ~ 0
+Text GLabel 7950 3650 2    50   Input ~ 0
 D+
-Text GLabel 7750 3650 2    50   Input ~ 0
+Text GLabel 7950 3750 2    50   Input ~ 0
 D-
 $Comp
@@
 Wire Wire Line
 	5550 1650 5600 1650
-Text Label 4500 2200 0    50   ~ 0
+Text Label 5550 2200 0    50   ~ 0
 RE_A
-Text Label 4500 2300 0    50   ~ 0
+Text Label 5550 2300 0    50   ~ 0
 RE_B
-Text Label 4500 2500 0    50   ~ 0
+Text Label 5550 2500 0    50   ~ 0
 ENC_S1
-Text Label 4500 2400 0    50   ~ 0
+Text Label 5550 2400 0    50   ~ 0
 ENC_S2
 $Comp
@@
 	8250 1900 7850 1900
 Connection ~ 7850 1900
+Wire Notes Line
+	7200 5550 26100 5550
+Wire Notes Line
+	26100 5550 26100 -9000
+Wire Wire Line
+	2400 3300 3300 3300
+$Comp
+L tinkerforge:SPST SW1
+U 1 1 5F612E1E
+P 2450 1800
+F 0 "SW1" H 2450 2065 50  0000 C CNN
+F 1 "SPST" H 2450 1974 50  0000 C CNN
+F 2 "Button_Switch_SMD:SW_SPST_REED_CT05-XXXX-G1" H 2450 1800 50  0001 C CNN
+F 3 "" H 2450 1800 50  0000 C CNN
+	1    2450 1800
+	1    0    0    -1
+$EndComp
+Wire Wire Line
+	2950 1500 2950 1800
+Connection ~ 2950 1800
+Wire Wire Line
+	2950 1800 2950 2200
+Wire Wire Line
+	4500 2200 5550 2200
+$Comp
+L Connector:AVR-ISP-6 J3
+U 1 1 5F656108
+P 6400 2550
+F 0 "J3" H 6070 2554 50  0000 R CNN
+F 1 "AVR-ISP-6" H 6070 2645 50  0000 R CNN
+F 2 "Connector_PinHeader_2.54mm:PinHeader_2x03_P2.54mm_Vertical" V 6150 2600 50  0001 C CNN
+F 3 " ~" H 5125 2000 50  0001 C CNN
+	1    6400 2550
+	-1   0    0    1
+$EndComp
+Text Label 3300 2200 2    50   ~ 0
+!RESET
+Text Label 2950 2200 2    50   ~ 0
+!RESET
+Text Label 5450 1900 2    50   ~ 0
+!RESET
+Wire Wire Line
+	6000 2450 6000 1900
+Wire Wire Line
+	6000 1900 5450 1900
+Wire Wire Line
+	4500 2500 5500 2500
+Wire Wire Line
+	4500 2400 5450 2400
+Wire Wire Line
+	4500 2300 5400 2300
+Wire Wire Line
+	5400 2300 5400 2550
+Wire Wire Line
+	5400 2550 6000 2550
+Connection ~ 5400 2300
+Wire Wire Line
+	5400 2300 5550 2300
+Wire Wire Line
+	5450 2400 5450 2650
+Wire Wire Line
+	5450 2650 6000 2650
+Connection ~ 5450 2400
+Wire Wire Line
+	5450 2400 5550 2400
+Wire Wire Line
+	5500 2500 5500 2750
+Wire Wire Line
+	5500 2750 6000 2750
+Connection ~ 5500 2500
+Wire Wire Line
+	5500 2500 5550 2500
+$Comp
+L power:+5V #PWR0118
+U 1 1 5F6A40D5
+P 6850 3050
+F 0 "#PWR0118" H 6850 2900 50  0001 C CNN
+F 1 "+5V" H 6865 3223 50  0000 C CNN
+F 2 "" H 6850 3050 50  0001 C CNN
+F 3 "" H 6850 3050 50  0001 C CNN
+	1    6850 3050
+	1    0    0    -1
+$EndComp
+Wire Wire Line
+	6850 3050 6500 3050
+$Comp
+L power:GND #PWR0119
+U 1 1 5F6A8DB1
+P 6950 2150
+F 0 "#PWR0119" H 6950 1900 50  0001 C CNN
+F 1 "GND" H 6955 1977 50  0000 C CNN
+F 2 "" H 6950 2150 50  0001 C CNN
+F 3 "" H 6950 2150 50  0001 C CNN
+	1    6950 2150
+	1    0    0    -1
+$EndComp
+Wire Wire Line
+	6950 2150 6500 2150
 $EndSCHEMATC
