File: kicad/macropad1.sch (KiCad schematic (older format))
At the start: 33 parts, among them J1 Conn_01x04, J2 USB_B_Mini, J3 AVR-ISP-6, P1 TestPoint, P20 TestPoint, P21 TestPoint, P28 TestPoint, P29 TestPoint, P30 TestPoint, P31 TestPoint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

Commit message: Adds iBom and final revision of board
Puts holes in the right place for the case
Adds proper backlight support with a properly sized mosfet (tiny)
Double checks dimensions
Parts:
- added H1, H2, H3, H4: MountingHole, MountingHole:MountingHole_2.7mm_M2.5, symbol Mechanical:MountingHole
Changed lines of the file:
@@
 Text Label 10100 1700 2    50   ~ 0
 PWM1
+$Comp
+L Mechanical:MountingHole H1
+U 1 1 5FBC66B9
+P 1000 7050
+F 0 "H1" H 1100 7096 50  0000 L CNN
+F 1 "MountingHole" H 1100 7005 50  0000 L CNN
+F 2 "MountingHole:MountingHole_2.7mm_M2.5" H 1000 7050 50  0001 C CNN
+F 3 "~" H 1000 7050 50  0001 C CNN
+	1    1000 7050
+	1    0    0    -1
+$EndComp
+$Comp
+L Mechanical:MountingHole H3
+U 1 1 5FBC7143
+P 1850 7050
+F 0 "H3" H 1950 7096 50  0000 L CNN
+F 1 "MountingHole" H 1950 7005 50  0000 L CNN
+F 2 "MountingHole:MountingHole_2.7mm_M2.5" H 1850 7050 50  0001 C CNN
+F 3 "~" H 1850 7050 50  0001 C CNN
+	1    1850 7050
+	1    0    0    -1
+$EndComp
+$Comp
+L Mechanical:MountingHole H4
+U 1 1 5FBC72DB
+P 1850 7300
+F 0 "H4" H 1950 7346 50  0000 L CNN
+F 1 "MountingHole" H 1950 7255 50  0000 L CNN
+F 2 "MountingHole:MountingHole_2.7mm_M2.5" H 1850 7300 50  0001 C CNN
+F 3 "~" H 1850 7300 50  0001 C CNN
+	1    1850 7300
+	1    0    0    -1
+$EndComp
+$Comp
+L Mechanical:MountingHole H2
+U 1 1 5FBC7533
+P 1000 7300
+F 0 "H2" H 1100 7346 50  0000 L CNN
+F 1 "MountingHole" H 1100 7255 50  0000 L CNN
+F 2 "MountingHole:MountingHole_2.7mm_M2.5" H 1000 7300 50  0001 C CNN
+F 3 "~" H 1000 7300 50  0001 C CNN
+	1    1000 7300
+	1    0    0    -1
+$EndComp
 $EndSCHEMATC
